File: hardware/sensorbuddy/sensors.kicad_sch (KiCad schematic)
At the start: 0 parts

Commit message: hardware: place parts for DryContact, PlugControl, SensorBuddy
Generate each board's schematic from a scripts/<board>.schgen.py manifest —
every part resolves to a real KiCad symbol + matching footprint + 3D model + LCSC.
Parts are PLACED, not wired (wire in eeschema; each sheet carries a pinout note).
make check-<board> = structure sound for all three:
- DryContact  (NEW): 49 components — STM32G0B1 + TCAN1044 + ULN2003 + 4x Omron
  G6K-2F-Y Form-C dry contacts; 29-bit CAN, UID auto-address. + BOM + handsolder.
- PlugControl (NEW KiCad project): 88 components — mcu/safety/actuation. A few
  generic stand-in symbols (TLV3202/74HC08/REF3330/TPS3823/SSR) pending swap;
  footprints/LCSC are correct.
- SensorBuddy (regenerated from placeholders): 81 components — ESP32-S3 + STM32G0B1
  + isolated ADM3260/ADS1115/OPA2376 probe front-end + NTC/1-Wire/floats.
Reuses the existing custom symbols in lib/symbols/sensorbuddy.kicad_sym.

Co-Authored-By: Claude Opus 4.8 (1M context) <noreply@anthropic.com>
Parts:
- added C20, C21, C33, C34: 100pF, Capacitor_SMD:C_0603_1608Metric, symbol Device:C
- added C22, C23, C24, C26, C30, C31, C32, C35, C36, C37, C38: 100nF, Capacitor_SMD:C_0603_1608Metric, symbol Device:C
- added C25: 4.7uF, Capacitor_SMD:C_0805_2012Metric, symbol Device:C
- added J10: 1-Wire A, TerminalBlock_Phoenix:TerminalBlock_Phoenix_MPT-0,5-3-2.54_1x03_P2.54mm_Horizontal, symbol Connector_Generic:Conn_01x03
- added J11: 1-Wire B, TerminalBlock_Phoenix:TerminalBlock_Phoenix_MPT-0,5-3-2.54_1x03_P2.54mm_Horizontal, symbol Connector_Generic:Conn_01x03
- added J12: FLOAT1, TerminalBlock_Phoenix:TerminalBlock_Phoenix_MPT-0,5-2-2.54_1x02_P2.54mm_Horizontal, symbol Connector_Generic:Conn_01x02
- added J13: FLOAT2, TerminalBlock_Phoenix:TerminalBlock_Phoenix_MPT-0,5-2-2.54_1x02_P2.54mm_Horizontal, symbol Connector_Generic:Conn_01x02
- added J14: FLOAT3, TerminalBlock_Phoenix:TerminalBlock_Phoenix_MPT-0,5-2-2.54_1x02_P2.54mm_Horizontal, symbol Connector_Generic:Conn_01x02
- added J15: FLOAT4, TerminalBlock_Phoenix:TerminalBlock_Phoenix_MPT-0,5-2-2.54_1x02_P2.54mm_Horizontal, symbol Connector_Generic:Conn_01x02
- added J5: PROBE 1 BNC, Connector_Coaxial:BNC_Amphenol_B6252HB-NPP3G-50_Horizontal, symbol Connector:Conn_Coaxial
- added J6: PROBE 2 BNC, Connector_Coaxial:BNC_Amphenol_B6252HB-NPP3G-50_Horizontal, symbol Connector:Conn_Coaxial
- added J7: NTC1, TerminalBlock_Phoenix:TerminalBlock_Phoenix_MPT-0,5-2-2.54_1x02_P2.54mm_Horizontal, symbol Connector_Generic:Conn_01x02
- added J8: NTC2, TerminalBlock_Phoenix:TerminalBlock_Phoenix_MPT-0,5-2-2.54_1x02_P2.54mm_Horizontal, symbol Connector_Generic:Conn_01x02
- added J9: NTC3, TerminalBlock_Phoenix:TerminalBlock_Phoenix_MPT-0,5-2-2.54_1x02_P2.54mm_Horizontal, symbol Connector_Generic:Conn_01x02
- added R20, R21, R22, R23: 100k, Resistor_SMD:R_0603_1608Metric, symbol Device:R
- added R24, R25: 220R, Resistor_SMD:R_0603_1608Metric, symbol Device:R
- added R30, R31, R32: 10k, Resistor_SMD:R_0603_1608Metric, symbol Device:R
- added R33, R35: 4.7k, Resistor_SMD:R_0603_1608Metric, symbol Device:R
- added R34, R36: 100R, Resistor_SMD:R_0603_1608Metric, symbol Device:R
- added U7: ADM3260ARSZ, Package_SO:SSOP-20_3.9x8.7mm_P0.635mm, symbol sensorbuddy:ADM3260ARSZ
- added U8: ADS1115IDGST, Package_SO:VSSOP-10_3x3mm_P0.5mm, symbol sensorbuddy:ADS1115IDGST
- added U9: OPA2376AIDR, Package_SO:SOIC-8_3.9x4.9mm_P1.27mm, symbol sensorbuddy:OPA2376AIDR
Connections:
- new net: U7.10 (NC), U7.4 (GND1), U7.5 (NC), U7.6 (NC), U7.7 (NC), U7.8 (GND1), U7.9 (NC)
- new net GND2: U7.11 (GND2), U7.12 (NC), U7.13 (NC), U7.14 (GND2), U7.15 (NC), U7.16 (NC), U7.20 (GND2)
Other:
- note added: "SENSORS — isolated probes + NTC + 1-Wire + floats. PLACED, not wired. ISOLATION: U7 ADM3260 = bidirectional I2C isolator + isoPower. VDD1(5V)/GND1 = MCU side ; VISO/GNDISO = probe side (ISO_3V3). STM32 I2C1 (SCL/SDA) -> U7 side-1 -> side-2 -> U8 ADS1115 I2C (addr 0x48, ADDR->GND). C26 ISO decouple. PROBES (x2, isolated): BNC J5/J6 center -> bias midpoint (R20/R21, R22/R23 = 100k to VISO/GNDISO) -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"
- note removed: "Sensor Interfaces Isolated Probes (pH / ORP): ADM3260ARSZ I2C isolator + isoPower → ISO_3V3 domain OPA2376AIDR dual unity-gain buffer (2 channels) ADS1115IDGST 16-bit differential ADC AIN0/1: Probe A (BNC), AIN2/3: Probe B (BNC) Mid-rail bias: 2× 100kΩ 0.1% divider + 0.1µF per channel 220Ω + 100pF output filter per buffer channel NTC Thermistors (×3): 3.3V → 10kΩ 0.1% fixed → STM32 ADC (PA0/PA1/P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"
- company: (none) -> blueAcro / ReefVolt
- title: ReefVolt SensorBuddy — Sensor Interfaces -> ReefVolt SensorBuddy — Main — Isolated pH/ORP probes (ADM3260+ADS1115+OPA2376), NTC, 1-Wire, floats
